Commit message: Camera and lidar sensor

File: description/common_properties.xacro (robot description, xacro)
@@ -9,4 +9,7 @@
     <material name="blue">
         <color rgba="0.2 0.2 1 1" />
+    </material>
+    <material name="red">
+        <color rgba="1 0 0 1" />
     </material>
     <material name="black">

File: description/robot.urdf.xacro (robot description, xacro)
@@ -4,3 +4,5 @@
     <xacro:include filename="robot_core.xacro" />
     <xacro:include filename="robot_core_gazebo.xacro" />
+    <xacro:include filename="lidar.xacro" />
+    <xacro:include filename="camera.xacro" />
 </robot>
